File: PCB/PCB.kicad_pcb (KiCad board)
At the start: 2 copper layers, 112.3 x 136.7 mm, 117 parts, among them J1 Conn_01x03_Pin, J10 Conn_01x03_Pin, J11 Conn_01x03_Pin, J12 Conn_01x03_Pin, J13 Conn_01x03_Pin, J14 Conn_01x03_Pin, J15 Conn_01x03_Pin, J16 Conn_01x03_Pin, J17 Conn_01x03_Pin, J18 Conn_01x03_Pin, J19 Conn_01x03_Pin, J2 Conn_01x03_Pin, J20 Conn_01x03_Pin, J21 Conn_01x03_Pin, J22 Conn_01x03_Pin, J23 Conn_01x03_Pin, J24 Conn_01x03_Pin, J25 Conn_01x03_Pin, J26 Conn_01x03_Pin, J27 Conn_01x03_Pin, J28 Conn_01x03_Pin, J29 Conn_01x03_Pin, J3 Conn_01x03_Pin, J30 Conn_01x03_Pin, J31 Conn_01x03_Pin, J32 Conn_01x03_Pin, J4 Conn_01x03_Pin, J5 Conn_01x03_Pin, J6 Conn_01x03_Pin, J7 Conn_01x03_Pin, J8 Conn_01x03_Pin, J9 Conn_01x03_Pin, P1 J1B1211CCD, U1 Teensy4.1, U2 74AHCT595, U3 74HCT245, U4 74AHCT595, U5 74HCT245, U6 74AHCT595, U7 74HCT245, U8 74AHCT595, U9 74HCT245

Commit message: update
Parts:
- moved LED_PWR_IN1 1.02 mm to (69.5, 23.5)
Routing:
- net /LED_R 1 to 8/LED_B_1: track 10.4 -> 12.8 mm
- net /LED_R 1 to 8/LED_R_1: track 42.7 -> 43.9 mm
Changed lines of the file:
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@@
   )
   (footprint "Connector_Wago:Wago_734-162_1x02_P3.50mm_Horizontal" (layer "F.Cu")
-    (at 69.464 24.47 180)
+    (at 69.464 23.454 180)
     (descr "Molex 734 Male header (for PCBs); Angled solder pin 1 x 1 mm, 734-162 , 2 Pins (http://www.farnell.com/datasheets/2157639.pdf), generated with kicad-footprint-generator")
     (tags "connector Wago  top entry")
@@
     )
   )
+  (gr_rect (start 28.448 17.018) (end 67.564 25.9334)
+    (stroke (width 0.15) (type solid)) (fill solid) (layer "B.Mask"))
+  (gr_rect (start 67.183 17.1323) (end 72.771 21.2217)
+    (stroke (width 0.15) (type solid)) (fill solid) (layer "B.Mask"))
+  (gr_rect (start 72.644 17.018) (end 109.982 25.9334)
+    (stroke (width 0.15) (type solid)) (fill solid) (layer "B.Mask"))
+  (gr_rect (start 28.448 17.018) (end 37.338 122.428)
+    (stroke (width 0.15) (type solid)) (fill solid) (layer "B.Mask"))
+  (gr_rect (start 101.092 17.399) (end 109.982 122.809)
+    (stroke (width 0.15) (type solid)) (fill solid) (layer "B.Mask"))
   (gr_rect (start 13.716 13.716) (end 125.984 150.368)
     (stroke (width 0.1) (type default)) (fill none) (layer "Edge.Cuts"))
@@
   (segment (start 105.156 38.608) (end 111.1264 38.608) (width 0.25) (layer "F.Cu") (net 53))
   (segment (start 111.1264 38.608) (end 114.1437 41.6253) (width 0.25) (layer "F.Cu") (net 53))
-  (segment (start 90.424 27.432) (end 97.271 20.585) (width 0.25) (layer "F.Cu") (net 54))
-  (segment (start 97.271 20.585) (end 97.9695 20.585) (width 0.25) (layer "F.Cu") (net 54))
-  (segment (start 97.9695 23.185) (end 96.715 23.185) (width 0.25) (layer "F.Cu") (net 55))
-  (segment (start 96.715 23.185) (end 95.9 24) (width 0.25) (layer "F.Cu") (net 55))
+  (segment (start 96.774 21.2805) (end 97.4695 20.585) (width 0.25) (layer "F.Cu") (net 54))
+  (segment (start 94.742 27.432) (end 95.358 26.816) (width 0.25) (layer "F.Cu") (net 54))
+  (segment (start 97.4695 20.585) (end 97.9695 20.585) (width 0.25) (layer "F.Cu") (net 54))
+  (segment (start 95.358 25.230814) (end 96.774 23.814814) (width 0.25) (layer "F.Cu") (net 54))
+  (segment (start 90.424 27.432) (end 94.742 27.432) (width 0.25) (layer "F.Cu") (net 54))
+  (segment (start 95.358 26.816) (end 95.358 25.230814) (width 0.25) (layer "F.Cu") (net 54))
+  (segment (start 96.774 23.814814) (end 96.774 21.2805) (width 0.25) (layer "F.Cu") (net 54))
+  (segment (start 95.758 25.3965) (end 97.9695 23.185) (width 0.25) (layer "F.Cu") (net 55))
+  (segment (start 95.758 27.432) (end 95.758 25.3965) (width 0.25) (layer "F.Cu") (net 55))
   (segment (start 86.2 58.8) (end 84.715 58.8) (width 0.25) (layer "F.Cu") (net 55))
   (via (at 86.2 58.8) (size 0.8) (drill 0.4) (layers "F.Cu" "B.Cu") (net 55))
-  (via (at 95.9 24) (size 0.8) (drill 0.4) (layers "F.Cu" "B.Cu") (net 55))
+  (via (at 95.758 27.432) (size 0.8) (drill 0.4) (layers "F.Cu" "B.Cu") (net 55))
   (segment (start 86.3 33.6) (end 86.3 58.7) (width 0.25) (layer "B.Cu") (net 55))
+  (segment (start 95.758 27.432) (end 92.468 27.432) (width 0.25) (layer "B.Cu") (net 55))
   (segment (start 86.3 58.7) (end 86.2 58.8) (width 0.25) (layer "B.Cu") (net 55))
-  (segment (start 95.9 24) (end 86.3 33.6) (width 0.25) (layer "B.Cu") (net 55))
+  (segment (start 92.468 27.432) (end 86.3 33.6) (width 0.25) (layer "B.Cu") (net 55))
   (segment (start 90.1015 80.6474) (end 96.9485 73.8004) (width 0.25) (layer "F.Cu") (net 56))
   (segment (start 96.9485 73.8004) (end 97.647 73.8004) (width 0.25) (layer "F.Cu") (net 56))
@@
   (segment (start 41.1 39.322) (end 41.1 31) (width 0.25) (layer "B.Cu") (net 75))
   (segment (start 41.875 30.225) (end 43.179 30.225) (width 0.25) (layer "B.Cu") (net 75))
-  (segment (start 92.7479 26.8581) (end 97.9695 26.8581) (width 0.25) (layer "F.Cu") (net 76))
-  (segment (start 90.424 29.182) (end 92.7479 26.8581) (width 0.25) (layer "F.Cu") (net 76))
+  (segment (start 96.1336 28.194) (end 97.4695 26.8581) (width 0.25) (layer "F.Cu") (net 76))
+  (segment (start 91.412 28.194) (end 96.1336 28.194) (width 0.25) (layer "F.Cu") (net 76))
+  (segment (start 90.424 29.182) (end 91.412 28.194) (width 0.25) (layer "F.Cu") (net 76))
+  (segment (start 97.4695 26.8581) (end 97.9695 26.8581) (width 0.25) (layer "F.Cu") (net 76))
   (segment (start 97.9695 29.4581) (end 96.5419 29.4581) (width 0.25) (layer "F.Cu") (net 77))
   (segment (start 92.8954 61.1046) (end 92.8954 60.5102) (width 0.25) (layer "F.Cu") (net 77))
@@
     )
   )
+  (zone (net 17) (net_name "GND") (layers "F&B.Cu") (hatch edge 0.5)
+    (priority 3)
+    (connect_pads (clearance 0.5))
+    (min_thickness 0.25) (filled_areas_thickness no)
+    (fill yes (thermal_gap 0.5) (thermal_bridge_width 1.5) (island_removal_mode 2) (island_area_min 10))
+    (polygon
+      (pts
+        (xy 68.072 21.844)
+        (xy 68.072 27.94)
+        (xy 71.12 27.94)
+        (xy 71.12 21.844)
+      )
+    )
+  )
   (zone (net 19) (net_name "+12V") (layer "B.Cu") (hatch edge 0.5)
-    (priority 1)
+    (priority 2)
     (connect_pads (clearance 0.5))
     (min_thickness 0.25) (filled_areas_thickness no)
-    (fill yes (thermal_gap 0.5) (thermal_bridge_width 0.5))
+    (fill yes (thermal_gap 0.5) (thermal_bridge_width 1.5) (island_removal_mode 2) (island_area_min 10))
     (polygon
       (pts
@@
         (xy 27.94 123.19)
         (xy 38.1 123.19)
-        (xy 38.1 25.4)
-        (xy 100.33 25.4)
+        (xy 37.846 26.162)
+        (xy 100.076 26.162)
         (xy 100.33 123.19)
         (xy 110.49 123.19)
